File: RGBW-Controller.kicad_sch (KiCad schematic)
At the start: 24 parts, among them J1 Power, J2 RGBW, Q1 AO3400A, Q2 AO3400A, Q3 AO3400A, Q4 AO3400A, U1 ESP-12F

Commit message: updated footprint of C2 and C3
Parts:
- C2, C3: footprint Capacitor_SMD:C_0603_1608Metric_Pad1.08x0.95mm_HandSolder -> Capacitor_SMD:C_0805_2012Metric_Pad1.18x1.45mm_HandSolder
Other:
- company: (none) -> maxl95
- title: (none) -> RGBW-Controller
Changed lines of the file:
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@@
 (kicad_sch (version 20211123) (generator eeschema)
   (paper "A4")
+  (title_block
+    (title "RGBW-Controller")
+    (date "11.01.2022")
+    (rev "V2.0")
+    (company "maxl95")
+  )
   (junction (at 222.25 35.56) (diameter 0) (color 0 0 0 0)
   )
@@
       (effects (font (size 1.27 1.27)) (justify left))
     )
-    (property "Footprint" "Capacitor_SMD:C_0603_1608Metric_Pad1.08x0.95mm_HandSolder" (id 2) (at 63.1952 107.95 0)
+    (property "Footprint" "Capacitor_SMD:C_0805_2012Metric_Pad1.18x1.45mm_HandSolder" (id 2) (at 63.1952 107.95 0)
       (effects (font (size 1.27 1.27)) hide)
     )
@@
       (effects (font (size 1.27 1.27)) (justify left))
     )
-    (property "Footprint" "Capacitor_SMD:C_0603_1608Metric_Pad1.08x0.95mm_HandSolder" (id 2) (at 47.9552 107.95 0)
+    (property "Footprint" "Capacitor_SMD:C_0805_2012Metric_Pad1.18x1.45mm_HandSolder" (id 2) (at 47.9552 107.95 0)
       (effects (font (size 1.27 1.27)) hide)
     )
@@
     )
     (path "/d3670c69-cfd0-43c3-8979-f01c4da3ae4c"
-      (reference "C2") (unit 1) (value "100n") (footprint "Capacitor_SMD:C_0603_1608Metric_Pad1.08x0.95mm_HandSolder")
+      (reference "C2") (unit 1) (value "100n") (footprint "Capacitor_SMD:C_0805_2012Metric_Pad1.18x1.45mm_HandSolder")
     )
     (path "/360100e6-a009-48ac-843f-45670dfe259d"
-      (reference "C3") (unit 1) (value "100n") (footprint "Capacitor_SMD:C_0603_1608Metric_Pad1.08x0.95mm_HandSolder")
+      (reference "C3") (unit 1) (value "100n") (footprint "Capacitor_SMD:C_0805_2012Metric_Pad1.18x1.45mm_HandSolder")
     )
     (path "/5b001c74-406c-4093-b91d-b83460882081"
